File: pcb/matrix.sch (KiCad schematic (older format))
At the start: 142 parts

Commit message: Update PCB KiCAD project
Parts:
- removed D65: 1N4148, Diode_SMD:D_SOD-123, symbol Device:D
- removed MX67: 1u, MX_Only:MXOnly-1U-NoLED, symbol Switch:SW_SPST
- added MX71, MX73: 1.25u, MX_Only:MXOnly-1.25U-NoLED, symbol Switch:SW_SPST
- added MX74: 6.25u, MX_Only:MXOnly-6.25U-ReversedStabilizers-NoLED, symbol Switch:SW_SPST
- MX62, MX64: value 1.25u -> 1.5u; footprint MX_Only:MXOnly-1.25U-NoLED -> MX_Only:MXOnly-1.5U-NoLED
- MX63: value 1.25u -> 1u; footprint MX_Only:MXOnly-1.25U-NoLED -> MX_Only:MXOnly-1U-NoLED
- MX65: value 6.25u -> 7u; footprint MX_Only:MXOnly-6.25U-ReversedStabilizers-NoLED -> MX_Only:MXOnly-7U-ReversedStabilizers-NoLED
- MX66: value 1u -> 1.25u; footprint MX_Only:MXOnly-1U-NoLED -> MX_Only:MXOnly-1.25U-NoLED
- MX67: renamed from MX68; value 1u -> 1.5u; footprint MX_Only:MXOnly-1U-NoLED -> MX_Only:MXOnly-1.5U-NoLED
- MX72: value 1.5u -> 1.25u; footprint MX_Only:MXOnly-1.5U-NoLED -> MX_Only:MXOnly-1.25U-NoLED
- MX75: renamed from MX73; value 1.5u -> 1.25u; footprint MX_Only:MXOnly-1.5U-NoLED -> MX_Only:MXOnly-1.25U-NoLED
- renumbered D66 to D65, D67 to D66, D68 to D67, D69 to D68, MX69 to MX68, MX70 to MX69, MX71 to MX70
Connections:
- net COL0: now also MX71.2 (B)
- net COL1: now also MX72.2 (B)
- net COL2: now also MX73.2 (B)
- net COL6: now also MX74.2 (B)
- net COL9: no longer MX72.2 (B)
- net at D64.2 (A), MX66.1 (A): no longer MX72.1 (A)
- net at D63.2 (A), MX65.1 (A): now also MX74.1 (A)
- net at D62.2 (A), MX64.1 (A): now also MX73.1 (A)
- net at D61.2 (A), MX63.1 (A): now also MX72.1 (A)
- net at D60.2 (A), MX62.1 (A): now also MX71.1 (A)
Changed lines of the file:
@@
 	-1   0    0    -1
 $EndComp
-Wire Wire Line
-	7250 4350 7150 4350
 Text GLabel 1800 950  2    50   Input ~ 0
 COL0
@@
 	8250 5100 8350 5100
 Wire Wire Line
-	7250 5100 7250 4350
-Wire Wire Line
-	7150 5100 7250 5100
-Wire Wire Line
 	9900 1200 9900 1550
 Wire Wire Line
@@
 	-1   0    0    -1
 $EndComp
-$Comp
-L Switch:SW_SPST MX73
-U 1 1 5F4970B7
-P 8050 5100
-F 0 "MX73" H 8050 5335 50  0000 C CNN
-F 1 "1.5u" H 8050 5244 50  0000 C CNN
-F 2 "MX_Only:MXOnly-1.5U-NoLED" H 8050 5100 50  0001 C CNN
-F 3 "~" H 8050 5100 50  0001 C CNN
-	1    8050 5100
-	-1   0    0    -1
-$EndComp
-$Comp
-L Switch:SW_SPST MX72
-U 1 1 5F4970BD
-P 6950 5100
-F 0 "MX72" H 6950 5335 50  0000 C CNN
-F 1 "1.5u" H 6950 5244 50  0000 C CNN
-F 2 "MX_Only:MXOnly-1.5U-NoLED" H 6950 5100 50  0001 C CNN
-F 3 "~" H 6950 5100 50  0001 C CNN
-	1    6950 5100
-	-1   0    0    -1
-$EndComp
 Wire Wire Line
 	1800 2250 1800 2950
@@
 $EndComp
 $Comp
-L Device:D D69
+L Device:D D68
 U 1 1 5F4970D6
 P 10450 4500
-F 0 "D69" V 10500 4750 50  0000 R CNN
+F 0 "D68" V 10500 4750 50  0000 R CNN
 F 1 "1N4148" V 10400 4850 50  0000 R CNN
 F 2 "Diode_SMD:D_SOD-123" H 10450 4500 50  0001 C CNN
@@
 $EndComp
 $Comp
-L Switch:SW_SPST MX71
+L Switch:SW_SPST MX70
 U 1 1 5F4970DC
 P 10250 4350
-F 0 "MX71" H 10250 4585 50  0000 C CNN
+F 0 "MX70" H 10250 4585 50  0000 C CNN
 F 1 "1u" H 10250 4494 50  0000 C CNN
 F 2 "MX_Only:MXOnly-1U-NoLED" H 10250 4350 50  0001 C CNN
@@
 Connection ~ 9350 4650
 $Comp
-L Device:D D68
+L Device:D D67
 U 1 1 5F4970E5
 P 9350 4500
-F 0 "D68" V 9400 4750 50  0000 R CNN
+F 0 "D67" V 9400 4750 50  0000 R CNN
 F 1 "1N4148" V 9300 4850 50  0000 R CNN
 F 2 "Diode_SMD:D_SOD-123" H 9350 4500 50  0001 C CNN
@@
 $EndComp
 $Comp
-L Switch:SW_SPST MX70
+L Switch:SW_SPST MX69
 U 1 1 5F4970EB
 P 9150 4350
-F 0 "MX70" H 9150 4585 50  0000 C CNN
+F 0 "MX69" H 9150 4585 50  0000 C CNN
 F 1 "1u" H 9150 4494 50  0000 C CNN
 F 2 "MX_Only:MXOnly-1U-NoLED" H 9150 4350 50  0001 C CNN
@@
 Connection ~ 8800 4650
 $Comp
-L Device:D D67
+L Device:D D66
 U 1 1 5F4970F4
 P 8800 4500
-F 0 "D67" V 8850 4750 50  0000 R CNN
+F 0 "D66" V 8850 4750 50  0000 R CNN
 F 1 "1N4148" V 8750 4850 50  0000 R CNN
 F 2 "Diode_SMD:D_SOD-123" H 8800 4500 50  0001 C CNN
@@
 $EndComp
 $Comp
-L Switch:SW_SPST MX69
+L Switch:SW_SPST MX68
 U 1 1 5F4970FA
 P 8600 4350
-F 0 "MX69" H 8600 4585 50  0000 C CNN
+F 0 "MX68" H 8600 4585 50  0000 C CNN
 F 1 "1u" H 8600 4494 50  0000 C CNN
 F 2 "MX_Only:MXOnly-1U-NoLED" H 8600 4350 50  0001 C CNN
@@
 Connection ~ 8250 4650
 $Comp
-L Device:D D66
+L Device:D D65
 U 1 1 5F497103
 P 8250 4500
-F 0 "D66" V 8300 4750 50  0000 R CNN
+F 0 "D65" V 8300 4750 50  0000 R CNN
 F 1 "1N4148" V 8200 4850 50  0000 R CNN
 F 2 "Diode_SMD:D_SOD-123" H 8250 4500 50  0001 C CNN
@@
 $EndComp
 Connection ~ 8250 4350
-Wire Wire Line
-	7850 4350 7850 5100
-Connection ~ 7850 4350
-$Comp
-L Switch:SW_SPST MX68
-U 1 1 5F49710C
-P 8050 4350
-F 0 "MX68" H 8050 4585 50  0000 C CNN
-F 1 "1u" H 8050 4494 50  0000 C CNN
-F 2 "MX_Only:MXOnly-1U-NoLED" H 8050 4350 50  0001 C CNN
-F 3 "~" H 8050 4350 50  0001 C CNN
-	1    8050 4350
-	-1   0    0    -1
-$EndComp
-Wire Wire Line
-	8250 4650 7700 4650
-Connection ~ 7700 4650
-$Comp
-L Device:D D65
-U 1 1 5F497115
-P 7700 4500
-F 0 "D65" V 7750 4750 50  0000 R CNN
-F 1 "1N4148" V 7650 4850 50  0000 R CNN
-F 2 "Diode_SMD:D_SOD-123" H 7700 4500 50  0001 C CNN
-F 3 "~" H 7700 4500 50  0001 C CNN
-F 4 "C81598" H 7700 4500 50  0001 C CNN "LCSC Part #"
-	1    7700 4500
-	0    -1   -1   0
-$EndComp
-$Comp
-L Switch:SW_SPST MX67
-U 1 1 5F49711B
-P 7500 4350
-F 0 "MX67" H 7500 4585 50  0000 C CNN
-F 1 "1u" H 7500 4494 50  0000 C CNN
-F 2 "MX_Only:MXOnly-1U-NoLED" H 7500 4350 50  0001 C CNN
-F 3 "~" H 7500 4350 50  0001 C CNN
-	1    7500 4350
-	-1   0    0    -1
-$EndComp
-Wire Wire Line
-	7700 4650 7150 4650
 Connection ~ 7150 4650
 $Comp
@@
 	0    -1   -1   0
 $EndComp
-Connection ~ 7150 4350
-Wire Wire Line
-	6750 5100 6750 4350
-Connection ~ 6750 4350
-$Comp
-L Switch:SW_SPST MX66
-U 1 1 5F49712D
-P 6950 4350
-F 0 "MX66" H 6950 4585 50  0000 C CNN
-F 1 "1u" H 6950 4494 50  0000 C CNN
-F 2 "MX_Only:MXOnly-1U-NoLED" H 6950 4350 50  0001 C CNN
-F 3 "~" H 6950 4350 50  0001 C CNN
-	1    6950 4350
-	-1   0    0    -1
-$EndComp
 Wire Wire Line
 	7150 4650 5500 4650
@@
 	0    -1   -1   0
 $EndComp
-$Comp
-L Switch:SW_SPST MX65
-U 1 1 5F49713C
-P 5300 4350
-F 0 "MX65" H 5300 4585 50  0000 C CNN
-F 1 "6.25u" H 5300 4494 50  0000 C CNN
-F 2 "MX_Only:MXOnly-6.25U-ReversedStabilizers-NoLED" H 5300 4350 50  0001 C CNN
-F 3 "~" H 5300 4350 50  0001 C CNN
-	1    5300 4350
-	-1   0    0    -1
-$EndComp
 Wire Wire Line
 	5500 4650 3300 4650
@@
 	0    -1   -1   0
 $EndComp
-$Comp
-L Switch:SW_SPST MX64
-U 1 1 5F49714B
-P 3100 4350
-F 0 "MX64" H 3100 4585 50  0000 C CNN
-F 1 "1.25u" H 3100 4494 50  0000 C CNN
-F 2 "MX_Only:MXOnly-1.25U-NoLED" H 3100 4350 50  0001 C CNN
-F 3 "~" H 3100 4350 50  0001 C CNN
-	1    3100 4350
-	-1   0    0    -1
-$EndComp
 Wire Wire Line
 	3300 4650 2750 4650
@@
 	0    -1   -1   0
 $EndComp
-$Comp
-L Switch:SW_SPST MX63
-U 1 1 5F49715A
-P 2550 4350
-F 0 "MX63" H 2550 4585 50  0000 C CNN
-F 1 "1.25u" H 2550 4494 50  0000 C CNN
-F 2 "MX_Only:MXOnly-1.25U-NoLED" H 2550 4350 50  0001 C CNN
-F 3 "~" H 2550 4350 50  0001 C CNN
-	1    2550 4350
-	-1   0    0    -1
-$EndComp
 Wire Wire Line
 	950  4650 2200 4650
@@
 $EndComp
 $Comp
-L Switch:SW_SPST MX62
-U 1 1 5F49716A
-P 2000 4350
-F 0 "MX62" H 2000 4585 50  0000 C CNN
-F 1 "1.25u" H 2000 4494 50  0000 C CNN
-F 2 "MX_Only:MXOnly-1.25U-NoLED" H 2000 4350 50  0001 C CNN
-F 3 "~" H 2000 4350 50  0001 C CNN
-	1    2000 4350
-	-1   0    0    -1
-$EndComp
-$Comp
 L Device:D D59
 U 1 1 5F497171
@@
 	0    -1   -1   0
 $EndComp
-Wire Wire Line
-	7300 3650 7300 4350
-Connection ~ 7300 3650
 $Comp
 L Switch:SW_SPST MX57
@@
 	-1   0    0    -1
 $EndComp
+Connection ~ 7850 4350
+Wire Wire Line
+	7850 4350 7850 5100
+Wire Wire Line
+	7150 4650 8250 4650
+$Comp
+L Switch:SW_SPST MX74
+U 1 1 5FB4808E
+P 5300 5050
+F 0 "MX74" H 5300 5285 50  0000 C CNN
+F 1 "6.25u" H 5300 5194 50  0000 C CNN
+F 2 "MX_Only:MXOnly-6.25U-ReversedStabilizers-NoLED" H 5300 5050 50  0001 C CNN
+F 3 "~" H 5300 5050 50  0001 C CNN
+	1    5300 5050
+	-1   0    0    -1
+$EndComp
+Wire Wire Line
+	5100 4350 5100 5050
+Connection ~ 5100 4350
+Wire Wire Line
+	5500 5050 5600 5050
+Wire Wire Line
+	5600 5050 5600 4350
+Wire Wire Line
+	5600 4350 5500 4350
+Connection ~ 5500 4350
+$Comp
+L Switch:SW_SPST MX71
+U 1 1 5FB57EAA
+P 2000 5050
+F 0 "MX71" H 2000 5285 50  0000 C CNN
+F 1 "1.25u" H 2000 5194 50  0000 C CNN
+F 2 "MX_Only:MXOnly-1.25U-NoLED" H 2000 5050 50  0001 C CNN
+F 3 "~" H 2000 5050 50  0001 C CNN
+	1    2000 5050
+	-1   0    0    -1
+$EndComp
+$Comp
+L Switch:SW_SPST MX73
+U 1 1 5FB58D92
+P 3100 5050
+F 0 "MX73" H 3100 5285 50  0000 C CNN
+F 1 "1.25u" H 3100 5194 50  0000 C CNN
+F 2 "MX_Only:MXOnly-1.25U-NoLED" H 3100 5050 50  0001 C CNN
+F 3 "~" H 3100 5050 50  0001 C CNN
+	1    3100 5050
+	-1   0    0    -1
+$EndComp
+$Comp
+L Switch:SW_SPST MX72
+U 1 1 5FB591B2
+P 2550 5050
+F 0 "MX72" H 2550 5285 50  0000 C CNN
+F 1 "1.25u" H 2550 5194 50  0000 C CNN
+F 2 "MX_Only:MXOnly-1.25U-NoLED" H 2550 5050 50  0001 C CNN
+F 3 "~" H 2550 5050 50  0001 C CNN
+	1    2550 5050
+	-1   0    0    -1
+$EndComp
+Wire Wire Line
+	1800 4350 1800 5050
+Connection ~ 1800 4350
+Wire Wire Line
+	2200 5050 2300 5050
+Wire Wire Line
+	2300 5050 2300 4350
+Wire Wire Line
+	2300 4350 2200 4350
+Connection ~ 2200 4350
+Wire Wire Line
+	2350 4350 2350 5050
+Connection ~ 2350 4350
+Wire Wire Line
+	2750 5050 2850 5050
+Wire Wire Line
+	2850 5050 2850 4350
+Wire Wire Line
+	2850 4350 2750 4350
+Connection ~ 2750 4350
+Wire Wire Line
+	2900 4350 2900 5050
+Connection ~ 2900 4350
+Wire Wire Line
+	3300 5050 3400 5050
+Wire Wire Line
+	3400 5050 3400 4350
+Wire Wire Line
+	3400 4350 3300 4350
+Connection ~ 3300 4350
+$Comp
+L Switch:SW_SPST MX62
+U 1 1 5F49716A
+P 2000 4350
+F 0 "MX62" H 2000 4585 50  0000 C CNN
+F 1 "1.5u" H 2000 4494 50  0000 C CNN
+F 2 "MX_Only:MXOnly-1.5U-NoLED" H 2000 4350 50  0001 C CNN
+F 3 "~" H 2000 4350 50  0001 C CNN
+	1    2000 4350
+	-1   0    0    -1
+$EndComp
+$Comp
+L Switch:SW_SPST MX63
+U 1 1 5F49715A
+P 2550 4350
+F 0 "MX63" H 2550 4585 50  0000 C CNN
+F 1 "1u" H 2550 4494 50  0000 C CNN
+F 2 "MX_Only:MXOnly-1U-NoLED" H 2550 4350 50  0001 C CNN
+F 3 "~" H 2550 4350 50  0001 C CNN
+	1    2550 4350
+	-1   0    0    -1
+$EndComp
+$Comp
+L Switch:SW_SPST MX64
+U 1 1 5F49714B
+P 3100 4350
+F 0 "MX64" H 3100 4585 50  0000 C CNN
+F 1 "1.5u" H 3100 4494 50  0000 C CNN
+F 2 "MX_Only:MXOnly-1.5U-NoLED" H 3100 4350 50  0001 C CNN
+F 3 "~" H 3100 4350 50  0001 C CNN
+	1    3100 4350
+	-1   0    0    -1
+$EndComp
+$Comp
+L Switch:SW_SPST MX65
+U 1 1 5F49713C
+P 5300 4350
+F 0 "MX65" H 5300 4585 50  0000 C CNN
+F 1 "7u" H 5300 4494 50  0000 C CNN
+F 2 "MX_Only:MXOnly-7U-ReversedStabilizers-NoLED" H 5300 4350 50  0001 C CNN
+F 3 "~" H 5300 4350 50  0001 C CNN
+	1    5300 4350
+	-1   0    0    -1
+$EndComp
+$Comp
+L Switch:SW_SPST MX75
+U 1 1 5F4970B7
+P 8050 5100
+F 0 "MX75" H 8050 5335 50  0000 C CNN
+F 1 "1.25u" H 8050 5244 50  0000 C CNN
+F 2 "MX_Only:MXOnly-1.25U-NoLED" H 8050 5100 50  0001 C CNN
+F 3 "~" H 8050 5100 50  0001 C CNN
+	1    8050 5100
+	-1   0    0    -1
+$EndComp
+$Comp
+L Switch:SW_SPST MX67
+U 1 1 5F49710C
+P 8050 4350
+F 0 "MX67" H 8050 4585 50  0000 C CNN
+F 1 "1.5u" H 8050 4494 50  0000 C CNN
+F 2 "MX_Only:MXOnly-1.5U-NoLED" H 8050 4350 50  0001 C CNN
+F 3 "~" H 8050 4350 50  0001 C CNN
+	1    8050 4350
+	-1   0    0    -1
+$EndComp
+$Comp
+L Switch:SW_SPST MX66
+U 1 1 5F49712D
+P 6950 4350
+F 0 "MX66" H 6950 4585 50  0000 C CNN
+F 1 "1.25u" H 6950 4494 50  0000 C CNN
+F 2 "MX_Only:MXOnly-1.25U-NoLED" H 6950 4350 50  0001 C CNN
+F 3 "~" H 6950 4350 50  0001 C CNN
+	1    6950 4350
+	-1   0    0    -1
+$EndComp
